File: hardware/MIDI Box.kicad_sch (KiCad schematic)
At the start: 31 parts, among them J1 Conn_01x02_Pin, J2 Conn_01x02_Pin, J3 Conn_01x20_Socket, J4 Conn_01x20_Socket, J5 MIDI_IN, J6 MIDI_OUT, J7 Conn_01x012_Pin, U1 6N138, U2 6N138, U3 40106

Commit message: v2.0 board with TRS sockets
Parts:
- removed J1, J2: Conn_01x02_Pin, Connector_PinHeader_2.54mm:PinHeader_1x02_P2.54mm_Vertical, symbol Connector:Conn_01x02_Pin
- removed J5: MIDI_IN, symbol Connector:DIN-5_180degree
- removed J6: MIDI_OUT, symbol Connector:DIN-5_180degree
- removed J7: Conn_01x012_Pin, Connector_PinHeader_2.54mm:PinHeader_1x12_P2.54mm_Vertical, symbol Connector:Conn_01x12_Pin
- added J1: MIDI_IN_1, own_components:Audio Jack PJ-3136-B, symbol Connector_Audio:AudioJack3
- added J2: MIDI_IN_2, own_components:Audio Jack PJ-3136-B, symbol Connector_Audio:AudioJack3
- added J5: MIDI_OUT_1, own_components:Audio Jack PJ-3136-B, symbol Connector_Audio:AudioJack3
- added J6: MIDI_OUT_2, own_components:Audio Jack PJ-3136-B, symbol Connector_Audio:AudioJack3
- added J7: MIDI_OUT_3, own_components:Audio Jack PJ-3136-B, symbol Connector_Audio:AudioJack3
- added J8: MIDI_OUT_4, own_components:Audio Jack PJ-3136-B, symbol Connector_Audio:AudioJack3
- added J9: MIDI_OUT_5, own_components:Audio Jack PJ-3136-B, symbol Connector_Audio:AudioJack3
- added R15, R20: 220, Resistor_THT:R_Axial_DIN0204_L3.6mm_D1.6mm_P5.08mm_Horizontal, symbol Device:R
- renumbered R15 to R16, R16 to R17, R17 to R18, R18 to R19
Connections:
- net +5V: now also R20.1
- net GND: now also J5.S, J6.S, J7.S, J8.S, J9.S; no longer U3.13
- net UART0 RX: now also J4.19 (Pin_19), R10.2, R8.2; no longer J3.17 (Pin_17), R7.2, R9.2
- net UART0 TX: now also J4.20 (Pin_20); no longer J3.16 (Pin_16)
- net UART1 RX: now also R7.2, R9.2; no longer R10.2, R8.2
- net at R11.2: now also J5.T
- net at U3.11, U3.2, U3.3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: now also U3.13
- net at U3.12: now also R15.1
- net at R16.2: now also J5.R
- net at R19.2: now also J8.R
- net at R14.2: now also J8.T
- net at R18.2: now also J7.R
- net at R13.2: now also J7.T
- net at R17.2: now also J6.R
- net at R12.2: now also J6.T
- net MIDI_IN1_4: no longer names the net of R1.1
- net MIDI_IN1_4: now also J1.R
- net MIDI_IN1_5: no longer names the net of D1.2 (A), U1.3 (C2)
- net MIDI_IN1_5: now also J1.T
- net MIDI_IN2_4: no longer names the net of R2.1
- net MIDI_IN2_4: now also J2.R
- net MIDI_IN2_5: no longer names the net of D2.2 (A), U2.3 (C2)
- net MIDI_IN2_5: now also J2.T
- new net: J9.T, R15.2
- new net: J9.R, R20.2
Other:
- moved on the sheet: R11, R12, R13, R14, R16, R17, R18, R19, U3A, U3B, U3C, U3D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
